File: grapto-v3-pcb-right.kicad_pcb (KiCad board)
At the start: 2 copper layers, 150.1 x 129.9 mm, 86 parts, among them J1 USB_C_Receptacle_USB2.0, J2 USB_C_Receptacle_USB2.0, SW1 SW_Push, SW10 SW_Push, SW11 SW_Push, SW12 SW_Push, SW13 SW_Push, SW14 SW_Push, SW15 SW_Push, SW16 SW_Push, SW17 SW_Push, SW18 SW_Push, SW19 SW_Push, SW2 SW_Push, SW20 SW_Push, SW21 SW_Push, SW22 SW_Push, SW23 SW_Push, SW24 SW_Push, SW25 SW_Push, SW26 SW_Push, SW27 SW_Push, SW28 SW_Push, SW29 SW_Push, SW3 SW_Push, SW30 SW_Push, SW31 SW_SPST, SW4 SW_Push, SW5 SW_Push, SW6 SW_Push, SW7 SW_Push, SW8 SW_Push, SW9 SW_Push, U1 ATmega32U4-AU, Y1 Crystal_GND24

Commit message: First draft layout.
Parts:
- added REF**: KiCad-Logo_8mm_SilkScreen, Symbol:KiCad-Logo_8mm_SilkScreen, B.Cu at (157.8, 145.1)
- moved D26 10.4 mm to (119.1, 109.8)
- moved D25 7.31 mm to (83.7, 153.5)
- moved D30 3.36 mm to (81.5, 140.3), turned to 0 degrees
- moved D18 2.30 mm to (190.1, 125.7), turned to 270 degrees
- moved D12 2.20 mm to (190.2, 105.0), turned to 270 degrees
- moved D6 2.13 mm to (190.1, 85.9), turned to 270 degrees
Connections:
- U1 pad 25: /Sheet61884E9A/row0 -> /Sheet6188018D/row0
- U1 pad 26: /Sheet61884E9A/row1 -> /Sheet6188018D/row1
- U1 pad 27: /Sheet61884E9A/row2 -> /Sheet6188018D/row2
- U1 pad 28: /Sheet61884E9A/row3 -> /Sheet6188018D/row3
- U1 pad 29: /Sheet61884E9A/row4 -> /Sheet6188018D/row4
- U1 pad 36: /Sheet61884E9A/col5 -> /Sheet6188018D/col5
- U1 pad 37: /Sheet61884E9A/col4 -> /Sheet6188018D/col4
- U1 pad 38: /Sheet61884E9A/col3 -> /Sheet6188018D/col3
- U1 pad 39: /Sheet61884E9A/col2 -> /Sheet6188018D/col2
- U1 pad 40: /Sheet61884E9A/col1 -> /Sheet6188018D/col1
- U1 pad 41: /Sheet61884E9A/col0 -> /Sheet6188018D/col0
Routing:
- net /Sheet6188018D/col4: track 0.00 -> 207.1 mm, vias 0 -> 12
- net /Sheet6188018D/col5: track 14.5 -> 205.2 mm, vias 2 -> 6
- net /Sheet6188018D/col0: track 0.00 -> 189.7 mm, vias 0 -> 2
- net /Sheet6188018D/col3: track 0.00 -> 172.7 mm, vias 0 -> 10
- net /Sheet6188018D/col1: track 0.00 -> 170.4 mm, vias 0 -> 12
- net /Sheet6188018D/col2: track 0.00 -> 160.6 mm, vias 0 -> 12
- net /Sheet6188018D/row0: track 123.3 -> 233.6 mm, vias 0 -> 2
- net /Sheet6188018D/row1: track 123.5 -> 215.3 mm, vias 0 -> 2
- net /Sheet6188018D/row4: track 101.4 -> 190.1 mm, vias 2 -> 4
- net /Sheet6188018D/row2: track 124.4 -> 209.6 mm, vias 0 -> 2
- net 0V: track 8.13 -> 70.8 mm, vias 27 -> 31
- net /Sheet6188018D/row3: track 133.9 -> 189.9 mm, vias 0 -> 2
- net Net-(D26-Pad1): track 0.00 -> 10.4 mm
- net Net-(D20-Pad1): track 0.00 -> 8.66 mm
- net Net-(D14-Pad1): track 0.00 -> 8.47 mm
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Other:
- board text added: "5v"
- board text added: "Grapto V3, Herman Lundkvist"
